Commit message: ...

File: m2wr_description/urdf/m2wr.xacro (robot description, xacro)
@@ -25,5 +25,5 @@
                 <box size="0.5 0.3 0.07"/>
             </geometry>
-            <material name="blue"/>
+            <material name="orange"/>
         </visual>
         <!-- caster front -->

Commit message: ...

File: m2wr_description/urdf/m2wr.xacro (robot description, xacro)
@@ -2,5 +2,6 @@
 <robot name="m2wr" xmlns:xacro="http://www.ros.org/wiki/xacro">
     <!-- inludes -->
-    <xacro:include filename="$(find m2wr_description)/urdf/macros.xacro" />
+    <xacro:include filename="$(find m2wr_description)/urdf/m2wr.gazebo" />
+    <xacro:include filename="$(find m2wr_description)/urdf/wheel.xacro" />
     <xacro:include filename="$(find m2wr_description)/urdf/materials.xacro" />
     <!-- main body -->
@@ -52,4 +53,35 @@
         </visual>
     </link>
+    <!-- sensor : link -->
+    <link name="sensor_laser">
+        <!-- inertial -->
+        <inertial>
+          <origin xyz="0 0 0" rpy="0 0 0" />
+          <mass value="1" />
+          <xacro:cylinder_inertia mass="1" r="0.05" l="0.1" />
+        </inertial>
+        <!-- visual -->
+        <visual>
+            <origin xyz="0 0 0" rpy="0 0 0" />
+            <geometry>
+                <cylinder radius="0.05" length="0.1"/>
+            </geometry>
+            <material name="black" />
+        </visual>
+        <!-- collision -->
+        <collision>
+            <origin xyz="0 0 0" rpy="0 0 0"/>
+            <geometry>
+                <cylinder radius="0.05" length="0.1"/>
+            </geometry>
+        </collision>
+    </link>
+    <!-- sensor : joint -->
+    <joint name="joint_sensor_laser" type="fixed">
+        <origin xyz="0.15 0 0.05" rpy="0 0 0"/>
+        <parent link="link_chassis"/>
+        <child link="sensor_laser"/>
+    </joint>
+    <!-- left and right wheels -->
     <xacro:link_wheel name="link_right_wheel" />
     <xacro:joint_wheel name="joint_right_wheel" child="link_right_wheel" origin_xyz="-0.05 0.20 0" />

Commit message: ...

File: m2wr_description/urdf/m2wr.xacro (robot description, xacro)
@@ -22,5 +22,5 @@
         <!-- visual -->
         <visual>
-            <origin rpy="0 0 0" xyz="0 0 0"/>
+            <origin rpy="0 0 0" xyz="0 0 0.1"/>
             <geometry>
                 <box size="0.5 0.3 0.07"/>
@@ -30,7 +30,7 @@
         <!-- caster front -->
         <collision name="caster_front_collision">
-            <origin rpy=" 0 0 0" xyz="0.35 0 -0.05"/>
+            <origin rpy=" 0 0 0" xyz="0.35 0 -0.07"/>
             <geometry>
-                <sphere radius="0.05"/>
+                <sphere radius="0.02"/>
             </geometry>
             <surface>
@@ -85,6 +85,6 @@
     <!-- left and right wheels -->
     <xacro:link_wheel name="link_right_wheel" />
-    <xacro:joint_wheel name="joint_right_wheel" child="link_right_wheel" origin_xyz="-0.05 0.20 0" />
+    <xacro:joint_wheel name="joint_right_wheel" child="link_right_wheel" origin_xyz="-0.05 0.20 0.1" />
     <xacro:link_wheel name="link_left_wheel" />
-    <xacro:joint_wheel name="joint_left_wheel" child="link_left_wheel" origin_xyz="-0.05 -0.20 0" />
+    <xacro:joint_wheel name="joint_left_wheel" child="link_left_wheel" origin_xyz="-0.05 -0.20 0.1" />
 </robot>

Commit message: ...

File: m2wr_description/urdf/m2wr.xacro (robot description, xacro)
@@ -67,5 +67,5 @@
                 <cylinder radius="0.05" length="0.1"/>
             </geometry>
-            <material name="black" />
+            <material name="wight" />
         </visual>
         <!-- collision -->
@@ -85,6 +85,6 @@
     <!-- left and right wheels -->
     <xacro:link_wheel name="link_right_wheel" />
-    <xacro:joint_wheel name="joint_right_wheel" child="link_right_wheel" origin_xyz="-0.05 0.20 0.1" />
+    <xacro:joint_wheel name="joint_right_wheel" child="link_right_wheel" origin_xyz="-0.05 0.17 0.1" />
     <xacro:link_wheel name="link_left_wheel" />
-    <xacro:joint_wheel name="joint_left_wheel" child="link_left_wheel" origin_xyz="-0.05 -0.20 0.1" />
+    <xacro:joint_wheel name="joint_left_wheel" child="link_left_wheel" origin_xyz="-0.05 -0.17 0.1" />
 </robot>

Commit message: ...

File: m2wr_description/urdf/m2wr.xacro (robot description, xacro)
@@ -79,5 +79,5 @@
     <!-- sensor : joint -->
     <joint name="joint_sensor_laser" type="fixed">
-        <origin xyz="0.15 0 0.05" rpy="0 0 0"/>
+        <origin xyz="0 0 0.20" rpy="0 0 0"/>
         <parent link="link_chassis"/>
         <child link="sensor_laser"/>
@@ -85,6 +85,6 @@
     <!-- left and right wheels -->
     <xacro:link_wheel name="link_right_wheel" />
-    <xacro:joint_wheel name="joint_right_wheel" child="link_right_wheel" origin_xyz="-0.05 0.17 0.1" />
+    <xacro:joint_wheel name="joint_right_wheel" child="link_right_wheel" origin_xyz="-0.2 0.20 0.1" />
     <xacro:link_wheel name="link_left_wheel" />
-    <xacro:joint_wheel name="joint_left_wheel" child="link_left_wheel" origin_xyz="-0.05 -0.17 0.1" />
+    <xacro:joint_wheel name="joint_left_wheel" child="link_left_wheel" origin_xyz="-0.2 -0.20 0.1" />
 </robot>

Commit message: ...

File: m2wr_description/urdf/m2wr.xacro (robot description, xacro)
@@ -30,5 +30,5 @@
         <!-- caster front -->
         <collision name="caster_front_collision">
-            <origin rpy=" 0 0 0" xyz="0.35 0 -0.07"/>
+            <origin rpy=" 0 0 0" xyz="0.35 0 0.065"/>
             <geometry>
                 <sphere radius="0.02"/>
@@ -84,7 +84,11 @@
     </joint>
     <!-- left and right wheels -->
-    <xacro:link_wheel name="link_right_wheel" />
-    <xacro:joint_wheel name="joint_right_wheel" child="link_right_wheel" origin_xyz="-0.2 0.20 0.1" />
-    <xacro:link_wheel name="link_left_wheel" />
-    <xacro:joint_wheel name="joint_left_wheel" child="link_left_wheel" origin_xyz="-0.2 -0.20 0.1" />
+    <xacro:link_wheel name="link_back_right_wheel" />
+    <xacro:joint_wheel name="joint_back_right_wheel" child="link_back_right_wheel" origin_xyz="-0.2 0.20 0.1" />
+    <xacro:link_wheel name="link_back_left_wheel" />
+    <xacro:joint_wheel name="joint_back_left_wheel" child="link_back_left_wheel" origin_xyz="-0.2 -0.20 0.1" />
+    <xacro:link_wheel name="link_front_right_wheel" />
+    <xacro:joint_wheel name="joint_front_right_wheel" child="link_front_right_wheel" origin_xyz="0.2 0.20 0.1" />
+    <xacro:link_wheel name="link_front_left_wheel" />
+    <xacro:joint_wheel name="joint_front_left_wheel" child="link_front_left_wheel" origin_xyz="0.2 -0.20 0.1" />
 </robot>

File: m2wr_description/urdf/wheel.xacro (robot description, xacro)
@@ -11,5 +11,5 @@
             </inertial>
             <!-- collision -->
-            <collision name="link_right_wheel_collision">
+            <collision name="link_wheel_collision">
                 <origin rpy="0 1.5707 1.5707" xyz="0 0 0"/>
                 <geometry>

Commit message: ...

File: m2wr_description/urdf/m2wr.xacro (robot description, xacro)
@@ -47,7 +47,7 @@
         </collision>
         <visual name="caster_front_visual">
-            <origin rpy=" 0 0 0" xyz="0.2 0 -0.05"/>
+            <origin rpy=" 0 0 0" xyz="0.35 0 0.065"/>
             <geometry>
-                <sphere radius="0.05"/>
+                <sphere radius="0.02"/>
             </geometry>
         </visual>

Commit message: ...

File: m2wr_description/urdf/m2wr.xacro (robot description, xacro)
@@ -30,5 +30,5 @@
         <!-- caster front -->
         <collision name="caster_front_collision">
-            <origin rpy=" 0 0 0" xyz="0.35 0 0.065"/>
+            <origin rpy=" 0 0 0" xyz="0.0 0 0.065"/>
             <geometry>
                 <sphere radius="0.02"/>
@@ -47,5 +47,5 @@
         </collision>
         <visual name="caster_front_visual">
-            <origin rpy=" 0 0 0" xyz="0.35 0 0.065"/>
+            <origin rpy=" 0 0 0" xyz="0.0 0 0.065"/>
             <geometry>
                 <sphere radius="0.02"/>

Commit message: ...

File: m2wr_description/urdf/m2wr.xacro (robot description, xacro)
@@ -30,7 +30,7 @@
         <!-- caster front -->
         <collision name="caster_front_collision">
-            <origin rpy=" 0 0 0" xyz="0.0 0 0.065"/>
+            <origin rpy=" 0 0 0" xyz="0.1 0 0.065"/>
             <geometry>
-                <sphere radius="0.02"/>
+                <sphere radius="0.065"/>
             </geometry>
             <surface>
@@ -47,7 +47,7 @@
         </collision>
         <visual name="caster_front_visual">
-            <origin rpy=" 0 0 0" xyz="0.0 0 0.065"/>
+            <origin rpy=" 0 0 0" xyz="0.1 0 0.065"/>
             <geometry>
-                <sphere radius="0.02"/>
+                <sphere radius="0.065"/>
             </geometry>
         </visual>
@@ -84,11 +84,7 @@
     </joint>
     <!-- left and right wheels -->
-    <xacro:link_wheel name="link_back_right_wheel" />
-    <xacro:joint_wheel name="joint_back_right_wheel" child="link_back_right_wheel" origin_xyz="-0.2 0.20 0.1" />
-    <xacro:link_wheel name="link_back_left_wheel" />
-    <xacro:joint_wheel name="joint_back_left_wheel" child="link_back_left_wheel" origin_xyz="-0.2 -0.20 0.1" />
-    <xacro:link_wheel name="link_front_right_wheel" />
-    <xacro:joint_wheel name="joint_front_right_wheel" child="link_front_right_wheel" origin_xyz="0.2 0.20 0.1" />
-    <xacro:link_wheel name="link_front_left_wheel" />
-    <xacro:joint_wheel name="joint_front_left_wheel" child="link_front_left_wheel" origin_xyz="0.2 -0.20 0.1" />
+    <xacro:link_wheel name="link_right_wheel" />
+    <xacro:joint_wheel name="joint_right_wheel" child="link_right_wheel" origin_xyz="-0.07 0.20 0.1" />
+    <xacro:link_wheel name="link_left_wheel" />
+    <xacro:joint_wheel name="joint_left_wheel" child="link_left_wheel" origin_xyz="-0.07 -0.20 0.1" />
 </robot>

Commit message: ...

File: m2wr_description/urdf/m2wr.xacro (robot description, xacro)
@@ -29,27 +29,4 @@
         </visual>
         <!-- caster front -->
-        <collision name="caster_front_collision">
-            <origin rpy=" 0 0 0" xyz="0.1 0 0.065"/>
-            <geometry>
-                <sphere radius="0.065"/>
-            </geometry>
-            <surface>
-                <friction>
-                    <!-- frictionless between these two surface -->
-                    <ode>
-                        <mu>0</mu>
-                        <mu2>0</mu2>
-                        <slip1>1.0</slip1>
-                        <slip2>1.0</slip2>
-                    </ode>
-                </friction>
-            </surface>
-        </collision>
-        <visual name="caster_front_visual">
-            <origin rpy=" 0 0 0" xyz="0.1 0 0.065"/>
-            <geometry>
-                <sphere radius="0.065"/>
-            </geometry>
-        </visual>
     </link>
     <!-- sensor : link -->

Commit message: ...

File: m2wr_description/urdf/m2wr.xacro (robot description, xacro)
@@ -29,4 +29,27 @@
         </visual>
         <!-- caster front -->
+        <collision name="caster_front_collision">
+            <origin rpy=" 0 0 0" xyz="0.1 0 0.065"/>
+            <geometry>
+                <sphere radius="0.035"/>
+            </geometry>
+            <surface>
+                <friction>
+                    <!-- frictionless between these two surface -->
+                    <ode>
+                        <mu>0</mu>
+                        <mu2>0</mu2>
+                        <slip1>1.0</slip1>
+                        <slip2>1.0</slip2>
+                    </ode>
+                </friction>
+            </surface>
+        </collision>
+        <visual name="caster_front_visual">
+            <origin rpy=" 0 0 0" xyz="0.1 0 0.065"/>
+            <geometry>
+                <sphere radius="0.035"/>
+            </geometry>
+        </visual>
     </link>
     <!-- sensor : link -->
@@ -56,5 +79,5 @@
     <!-- sensor : joint -->
     <joint name="joint_sensor_laser" type="fixed">
-        <origin xyz="0 0 0.20" rpy="0 0 0"/>
+        <origin xyz="0 0 0.140" rpy="0 0 0"/>
         <parent link="link_chassis"/>
         <child link="sensor_laser"/>

Commit message: ...

File: m2wr_description/urdf/m2wr.xacro (robot description, xacro)
@@ -30,5 +30,5 @@
         <!-- caster front -->
         <collision name="caster_front_collision">
-            <origin rpy=" 0 0 0" xyz="0.1 0 0.065"/>
+            <origin rpy=" 0 0 0" xyz="0.1 0 -0.05"/>
             <geometry>
                 <sphere radius="0.035"/>
@@ -79,5 +79,5 @@
     <!-- sensor : joint -->
     <joint name="joint_sensor_laser" type="fixed">
-        <origin xyz="0 0 0.140" rpy="0 0 0"/>
+        <origin xyz="0 0 0.040" rpy="0 0 0"/>
         <parent link="link_chassis"/>
         <child link="sensor_laser"/>
@@ -85,6 +85,6 @@
     <!-- left and right wheels -->
     <xacro:link_wheel name="link_right_wheel" />
-    <xacro:joint_wheel name="joint_right_wheel" child="link_right_wheel" origin_xyz="-0.07 0.20 0.1" />
+    <xacro:joint_wheel name="joint_right_wheel" child="link_right_wheel" origin_xyz="-0.07 0.20 0.0" />
     <xacro:link_wheel name="link_left_wheel" />
-    <xacro:joint_wheel name="joint_left_wheel" child="link_left_wheel" origin_xyz="-0.07 -0.20 0.1" />
+    <xacro:joint_wheel name="joint_left_wheel" child="link_left_wheel" origin_xyz="-0.07 -0.20 0.0" />
 </robot>

Commit message: ...

File: m2wr_description/urdf/m2wr.xacro (robot description, xacro)
@@ -22,5 +22,5 @@
         <!-- visual -->
         <visual>
-            <origin rpy="0 0 0" xyz="0 0 0.1"/>
+            <origin rpy="0 0 0" xyz="0 0 0.0"/>
             <geometry>
                 <box size="0.5 0.3 0.07"/>
@@ -30,7 +30,7 @@
         <!-- caster front -->
         <collision name="caster_front_collision">
-            <origin rpy=" 0 0 0" xyz="0.1 0 -0.05"/>
+            <origin rpy=" 0 0 0" xyz="0.35 0 -0.05"/>
             <geometry>
-                <sphere radius="0.035"/>
+                <sphere radius="0.05"/>
             </geometry>
             <surface>
@@ -47,7 +47,7 @@
         </collision>
         <visual name="caster_front_visual">
-            <origin rpy=" 0 0 0" xyz="0.1 0 0.065"/>
+            <origin rpy=" 0 0 0" xyz="0.2 0 -0.05"/>
             <geometry>
-                <sphere radius="0.035"/>
+                <sphere radius="0.05"/>
             </geometry>
         </visual>
@@ -85,6 +85,6 @@
     <!-- left and right wheels -->
     <xacro:link_wheel name="link_right_wheel" />
-    <xacro:joint_wheel name="joint_right_wheel" child="link_right_wheel" origin_xyz="-0.07 0.20 0.0" />
+    <xacro:joint_wheel name="joint_right_wheel" child="link_right_wheel" origin_xyz="-0.05 0.20 0.0" />
     <xacro:link_wheel name="link_left_wheel" />
-    <xacro:joint_wheel name="joint_left_wheel" child="link_left_wheel" origin_xyz="-0.07 -0.20 0.0" />
+    <xacro:joint_wheel name="joint_left_wheel" child="link_left_wheel" origin_xyz="-0.05 -0.20 0.0" />
 </robot>

Commit message: ...

File: m2wr_description/urdf/m2wr.xacro (robot description, xacro)
@@ -52,4 +52,28 @@
             </geometry>
         </visual>
+        <!-- caster back -->
+        <collision name="caster_back_collision">
+            <origin rpy=" 0 0 0" xyz="-0.35 0 -0.05"/>
+            <geometry>
+                <sphere radius="0.05"/>
+            </geometry>
+            <surface>
+                <friction>
+                    <!-- frictionless between these two surface -->
+                    <ode>
+                        <mu>0</mu>
+                        <mu2>0</mu2>
+                        <slip1>1.0</slip1>
+                        <slip2>1.0</slip2>
+                    </ode>
+                </friction>
+            </surface>
+        </collision>
+        <visual name="caster_back_visual">
+            <origin rpy=" 0 0 0" xyz="-0.2 0 -0.05"/>
+            <geometry>
+                <sphere radius="0.05"/>
+            </geometry>
+        </visual>
     </link>
     <!-- sensor : link -->

Commit message: ...

File: m2wr_description/urdf/m2wr.xacro (robot description, xacro)
@@ -103,5 +103,5 @@
     <!-- sensor : joint -->
     <joint name="joint_sensor_laser" type="fixed">
-        <origin xyz="0 0 0.040" rpy="0 0 0"/>
+        <origin xyz="0 0 0.150" rpy="0 0 0"/>
         <parent link="link_chassis"/>
         <child link="sensor_laser"/>

Commit message: added: camera

File: m2wr_description/urdf/m2wr.xacro (robot description, xacro)
@@ -5,4 +5,15 @@
     <xacro:include filename="$(find m2wr_description)/urdf/wheel.xacro" />
     <xacro:include filename="$(find m2wr_description)/urdf/materials.xacro" />
+    <!-- hyper parameters : camera -->
+    <xacro:property name="camera_size" value="0.02"/>
+    <xacro:property name="camera_origin_x" value="0.15"/>
+    <xacro:property name="camera_origin_y" value="0"/>
+    <xacro:property name="camera_origin_z" value="0.05"/>
+    <xacro:macro name="default_inertial" params="mass">
+        <inertial>
+            <mass value="${mass}"/>
+            <inertia ixx="1.0" ixy="0.0" ixz="0.0" iyy="1.0" iyz="0.0" izz="1.0"/>
+        </inertial>
+    </xacro:macro>
     <!-- main body -->
     <link name="link_chassis">
@@ -78,32 +89,25 @@
     </link>
     <!-- sensor : link -->
-    <link name="sensor_laser">
-        <!-- inertial -->
-        <inertial>
-          <origin xyz="0 0 0" rpy="0 0 0" />
-          <mass value="1" />
-          <xacro:cylinder_inertia mass="1" r="0.05" l="0.1" />
-        </inertial>
+    <link name="camera">
         <!-- visual -->
         <visual>
-            <origin xyz="0 0 0" rpy="0 0 0" />
             <geometry>
-                <cylinder radius="0.05" length="0.1"/>
+                <box size="${camera_size} ${camera_size} ${camera_size}"/>
             </geometry>
-            <material name="wight" />
+        <material name="white"/>
         </visual>
-        <!-- collision -->
+        <!-- collsion -->
         <collision>
-            <origin xyz="0 0 0" rpy="0 0 0"/>
             <geometry>
-                <cylinder radius="0.05" length="0.1"/>
+                <box size="${camera_size} ${camera_size} ${camera_size}"/>
             </geometry>
         </collision>
+        <xacro:default_inertial mass="0.02"/>
     </link>
     <!-- sensor : joint -->
-    <joint name="joint_sensor_laser" type="fixed">
-        <origin xyz="0 0 0.150" rpy="0 0 0"/>
+    <joint name="camera_joint" type="fixed">
+        <origin xyz="${camera_origin_x} ${camera_origin_y} ${camera_origin_z}" rpy="0 0 0"/>
         <parent link="link_chassis"/>
-        <child link="sensor_laser"/>
+        <child link="camera"/>
     </joint>
     <!-- left and right wheels -->

Commit message: ...

File: m2wr_description/urdf/m2wr.xacro (robot description, xacro)
@@ -6,5 +6,5 @@
     <xacro:include filename="$(find m2wr_description)/urdf/materials.xacro" />
     <!-- hyper parameters : camera -->
-    <xacro:property name="camera_size" value="0.02"/>
+    <xacro:property name="camera_size" value="0.06"/>
     <xacro:property name="camera_origin_x" value="0.15"/>
     <xacro:property name="camera_origin_y" value="0"/>
@@ -93,5 +93,5 @@
         <visual>
             <geometry>
-                <box size="${camera_size} ${camera_size} ${camera_size}"/>
+                <box size="${camera_size/3} ${camera_size*2} ${camera_size/2}"/>
             </geometry>
         <material name="white"/>

Commit message: ...

File: m2wr_description/urdf/m2wr.xacro (robot description, xacro)
@@ -7,7 +7,7 @@
     <!-- hyper parameters : camera -->
     <xacro:property name="camera_size" value="0.06"/>
-    <xacro:property name="camera_origin_x" value="0.15"/>
+    <xacro:property name="camera_origin_x" value="0.24"/>
     <xacro:property name="camera_origin_y" value="0"/>
-    <xacro:property name="camera_origin_z" value="0.05"/>
+    <xacro:property name="camera_origin_z" value="0.06"/>
     <xacro:macro name="default_inertial" params="mass">
         <inertial>
@@ -93,5 +93,5 @@
         <visual>
             <geometry>
-                <box size="${camera_size/3} ${camera_size*2} ${camera_size/2}"/>
+                <box size="${camera_size/3} ${camera_size} ${camera_size/2}"/>
             </geometry>
         <material name="white"/>
@@ -100,5 +100,5 @@
         <collision>
             <geometry>
-                <box size="${camera_size} ${camera_size} ${camera_size}"/>
+                <box size="${camera_size/3} ${camera_size} ${camera_size/2}"/>
             </geometry>
         </collision>

Commit message: ...

File: m2wr_description/urdf/m2wr.xacro (robot description, xacro)
@@ -9,5 +9,5 @@
     <xacro:property name="camera_origin_x" value="0.24"/>
     <xacro:property name="camera_origin_y" value="0"/>
-    <xacro:property name="camera_origin_z" value="0.06"/>
+    <xacro:property name="camera_origin_z" value="0.05"/>
     <xacro:macro name="default_inertial" params="mass">
         <inertial>
@@ -100,5 +100,5 @@
         <collision>
             <geometry>
-                <box size="${camera_size/3} ${camera_size} ${camera_size/2}"/>
+                <box size="${{camera_size/3} ${camera_size} ${camera_size/2}"/>
             </geometry>
         </collision>

Commit message: ...

File: m2wr_description/urdf/m2wr.xacro (robot description, xacro)
@@ -100,5 +100,5 @@
         <collision>
             <geometry>
-                <box size="${{camera_size/3} ${camera_size} ${camera_size/2}"/>
+                <box size="${camera_size/3} ${camera_size} ${camera_size/2}"/>
             </geometry>
         </collision>
